Commit message: add new step to solve multi spawn

File: dr_description/description/camera.xacro (robot description, xacro)
@@ -1,4 +1,5 @@
 <?xml version="1.0"?>
 <robot xmlns:xacro="http://www.ros.org/wiki/xacro" >
+    <xacro:arg name="robot_namespace" default=""/>
     <joint name="camera_joint" type="fixed">
         <parent link="chassis"/>
@@ -46,4 +47,7 @@
             </camera>
             <plugin name="camera_controller" filename="libgazebo_ros_camera.so">
+                <ros>
+                    <namespace>${robot_namespace}</namespace>
+                </ros>
                 <frame_name>camera_link_optical</frame_name>
             </plugin>

File: dr_description/description/depth_camera2.xacro (robot description, xacro)
@@ -1,4 +1,5 @@
 <?xml version="1.0"?>
 <robot xmlns:xacro="http://www.ros.org/wiki/xacro" >
+    <xacro:macro name="depth_camera2" params="robot_namespace:=''">
     <joint name="scanner_joint" type="fixed">
         <parent link="chassis"/>
@@ -39,4 +40,7 @@
             </camera>
             <plugin name="scanner_controller" filename="libgazebo_ros_camera.so">
+                <ros>
+                    <namespace>${robot_namespace}</namespace>
+                </ros>
                 <frame_name>scanner_link_optical</frame_name>
                 <min_depth>0.1</min_depth>
@@ -45,3 +49,4 @@
         </sensor>
     </gazebo>
+    </xacro:macro>
 </robot>

File: dr_description/description/robot.urdf.xacro (robot description, xacro)
@@ -1,12 +1,24 @@
 <?xml version="1.0"?>
 <robot xmlns:xacro="http://www.ros.org/wiki/xacro"  name="robot">
+    <xacro:arg name="robot_namespace" default=""/>
+    <xacro:arg name="controllers_file" default=""/>
+    <xacro:arg name="ros2ctl_file" default=""/>
     <xacro:arg name="use_ros2_control" default="true"/>
     <xacro:arg name="sim_mode" default="false"/>
+    <xacro:property name="robot_namespace" value="$(arg robot_namespace)"/>
+    <xacro:property name="controllers_file" value="$(arg controllers_file)"/>
+    <xacro:property name="ros2ctl_file" value="$(arg ros2ctl_file)"/>
     <xacro:include filename="robot_core.xacro" />
     <xacro:if value="$(arg use_ros2_control)">
-        <xacro:include filename="ros2_control.xacro" />
+        <xacro:include filename="ros2_control.xacro"/>
+        <xacro:ros2_control
+            robot_namespace="${robot_namespace}"
+            controllers_file="${controllers_file}"
+            ros2ctl_file="${ros2ctl_file}"
+            sim_mode="$(arg sim_mode)"/>
     </xacro:if>
     <xacro:unless value="$(arg use_ros2_control)">
         <xacro:include filename="gazebo_control.xacro" />
+        <xacro:gazebo_control robot_namespace="${robot_namespace}" />
     </xacro:unless>
     <xacro:include filename="lidar.xacro" />
@@ -14,4 +26,7 @@
     <xacro:include filename="depth_camera.xacro" />
     <xacro:include filename="depth_camera2.xacro" />
+    <xacro:lidar            robot_namespace="${robot_namespace}" />
+    <xacro:depth_camera     robot_namespace="${robot_namespace}" />
+    <xacro:depth_camera2    robot_namespace="${robot_namespace}" />
     <!-- <xacro:include filename="face.xacro" /> -->
 </robot>

File: dr_description/description_1/camera.xacro (robot description, xacro)
@@ -1,9 +1,8 @@
 <?xml version="1.0"?>
 <robot xmlns:xacro="http://www.ros.org/wiki/xacro" >
-    <xacro:macro name="depth_camera" params="robot_namespace:=''">
     <joint name="camera_joint" type="fixed">
         <parent link="chassis"/>
         <child link="camera_link"/>
-        <origin xyz="0.305 0 0.08" rpy="0 0 0"/>
+        <origin xyz="0.276 0 0.181" rpy="0 0.18 0"/>
     </joint>
     <link name="camera_link">
@@ -12,5 +11,12 @@
                 <box size="0.010 0.03 0.03"/>
             </geometry>
-            <material name="red"/>
+            <material name="black"/>
+        </visual>
+        <visual>
+            <origin xyz="0 0 -0.05"/>
+            <geometry>
+                <cylinder radius="0.002" length="0.1"/>
+            </geometry>
+            <material name="black"/>
         </visual>
     </link>
@@ -22,6 +28,6 @@
     <link name="camera_link_optical"></link>
     <gazebo reference="camera_link">
-        <material>Gazebo/Red</material>
-        <sensor name="camera" type="depth">
+        <material>Gazebo/Black</material>
+        <sensor name="camera" type="camera">
             <pose> 0 0 0 0 0 0 </pose>
             <visualize>true</visualize>
@@ -30,5 +36,5 @@
                 <horizontal_fov>1.089</horizontal_fov>
                 <image>
-                    <format>B8G8R8</format>
+                    <format>R8G8B8</format>
                     <width>640</width>
                     <height>480</height>
@@ -40,13 +46,7 @@
             </camera>
             <plugin name="camera_controller" filename="libgazebo_ros_camera.so">
-                <ros>
-                    <namespace>${robot_namespace}</namespace>
-                </ros>
                 <frame_name>camera_link_optical</frame_name>
-                <min_depth>0.1</min_depth>
-                <max_depth>100.0</max_depth>
             </plugin>
         </sensor>
     </gazebo>
-    </xacro:macro>
 </robot>

File: dr_description/description_1/depth_camera.xacro (robot description, xacro)
@@ -1,5 +1,4 @@
 <?xml version="1.0"?>
 <robot xmlns:xacro="http://www.ros.org/wiki/xacro" >
-    <xacro:macro name="depth_camera" params="robot_namespace:=''">
     <joint name="camera_joint" type="fixed">
         <parent link="chassis"/>
@@ -40,7 +39,4 @@
             </camera>
             <plugin name="camera_controller" filename="libgazebo_ros_camera.so">
-                <ros>
-                    <namespace>${robot_namespace}</namespace>
-                </ros>
                 <frame_name>camera_link_optical</frame_name>
                 <min_depth>0.1</min_depth>
@@ -49,4 +45,3 @@
         </sensor>
     </gazebo>
-    </xacro:macro>
 </robot>

File: dr_description/description_1/depth_camera2.xacro (robot description, xacro)
@@ -1,11 +1,10 @@
 <?xml version="1.0"?>
 <robot xmlns:xacro="http://www.ros.org/wiki/xacro" >
-    <xacro:macro name="depth_camera" params="robot_namespace:=''">
-    <joint name="camera_joint" type="fixed">
+    <joint name="scanner_joint" type="fixed">
         <parent link="chassis"/>
-        <child link="camera_link"/>
-        <origin xyz="0.305 0 0.08" rpy="0 0 0"/>
+        <child link="scanner_link"/>
+        <origin xyz="0.1675 0.1325 0.08" rpy="0 0 1.5708"/>
     </joint>
-    <link name="camera_link">
+    <link name="scanner_link">
         <visual>
             <geometry>
@@ -15,13 +14,13 @@
         </visual>
     </link>
-    <joint name="camera_optical_joint" type="fixed">
-        <parent link="camera_link"/>
-        <child link="camera_link_optical"/>
+    <joint name="scanner_optical_joint" type="fixed">
+        <parent link="scanner_link"/>
+        <child link="scanner_link_optical"/>
         <origin xyz="0 0 0" rpy="${-pi/2} 0 ${-pi/2}"/>
     </joint>
-    <link name="camera_link_optical"></link>
-    <gazebo reference="camera_link">
+    <link name="scanner_link_optical"></link>
+    <gazebo reference="scanner_link">
         <material>Gazebo/Red</material>
-        <sensor name="camera" type="depth">
+        <sensor name="scanner" type="depth">
             <pose> 0 0 0 0 0 0 </pose>
             <visualize>true</visualize>
@@ -39,9 +38,6 @@
                 </clip>
             </camera>
-            <plugin name="camera_controller" filename="libgazebo_ros_camera.so">
-                <ros>
-                    <namespace>${robot_namespace}</namespace>
-                </ros>
-                <frame_name>camera_link_optical</frame_name>
+            <plugin name="scanner_controller" filename="libgazebo_ros_camera.so">
+                <frame_name>scanner_link_optical</frame_name>
                 <min_depth>0.1</min_depth>
                 <max_depth>100.0</max_depth>
@@ -49,4 +45,3 @@
         </sensor>
     </gazebo>
-    </xacro:macro>
 </robot>

File: dr_description/description_1/gazebo_control.xacro (robot description, xacro)
@@ -1,18 +1,6 @@
 <?xml version="1.0"?>
 <robot xmlns:xacro="http://www.ros.org/wiki/xacro">
-    <xacro:macro name="gazebo_control" params="robot_namespace:=''">
-    <xacro:if value="${robot_namespace != ''}">
-        <xacro:property name="odom_frame" value="${robot_namespace}/odom"/>
-        <xacro:property name="base_frame" value="${robot_namespace}/base_link"/>
-    </xacro:if>
-    <xacro:unless value="${robot_namespace != ''}">
-        <xacro:property name="odom_frame" value="odom"/>
-        <xacro:property name="base_frame" value="base_link"/>
-    </xacro:unless>
     <gazebo>
         <plugin name="diff_drive" filename="libgazebo_ros_diff_drive.so">
-            <ros>
-                <namespace>${robot_namespace}</namespace>
-            </ros>
             <!-- Wheel Information -->
             <left_joint>left_wheel_joint</left_joint>
@@ -24,6 +12,6 @@
             <max_wheel_acceleration>10.0</max_wheel_acceleration>
             <!-- Output -->
-            <odometry_frame>${odom_frame}</odometry_frame>
-            <robot_base_frame>${base_frame}</robot_base_frame>
+            <odometry_frame>odom</odometry_frame>
+            <robot_base_frame>base_link</robot_base_frame>
             <publish_odom>true</publish_odom>
             <publish_odom_tf>true</publish_odom_tf>
@@ -31,4 +19,3 @@
         </plugin>
     </gazebo>
-    </xacro:macro>
 </robot>

File: dr_description/description_1/lidar.xacro (robot description, xacro)
@@ -1,5 +1,4 @@
 <?xml version="1.0"?>
 <robot xmlns:xacro="http://www.ros.org/wiki/xacro" >
-    <xacro:macro name="lidar" params="robot_namespace:=''">
     <joint name="laser_joint" type="fixed">
         <parent link="chassis"/>
@@ -44,6 +43,5 @@
             <plugin name="laser_controller" filename="libgazebo_ros_ray_sensor.so">
                 <ros>
-                    <namespace>${robot_namespace}</namespace>
-                    <remapping>~/out:=scan</remapping>
+                    <argument>~/out:=scan</argument>
                 </ros>
                 <output_type>sensor_msgs/LaserScan</output_type>
@@ -52,4 +50,3 @@
         </sensor>
     </gazebo>
-    </xacro:macro>
 </robot>

File: dr_description/description_1/ros2_control.xacro (robot description, xacro)
@@ -1,6 +1,5 @@
 <?xml version="1.0"?>
 <robot xmlns:xacro="http://www.ros.org/wiki/xacro">
-    <xacro:macro name="ros2_control" params="robot_namespace controllers_file ros2ctl_file sim_mode">
-    <xacro:unless value="${sim_mode}">
+    <xacro:unless value="$(arg sim_mode)">
         <ros2_control name="RealRobot" type="system">
             <hardware>
@@ -32,5 +31,5 @@
         </ros2_control>
     </xacro:unless>
-    <xacro:if value="${sim_mode}">
+    <xacro:if value="$(arg sim_mode)">
         <ros2_control name="GazeboSystem" type="system">
             <hardware>
@@ -56,12 +55,8 @@
     </xacro:if>
     <gazebo>
-        <plugin name="${robot_namespace}_gazebo_ros2_control" filename="libgazebo_ros2_control.so">
-            <ros>
-                <namespace>${robot_namespace}</namespace>
-            </ros>
-            <parameters>${controllers_file}</parameters>
-            <parameters>${ros2ctl_file}</parameters>
+        <plugin name="gazebo_ros2_control" filename="libgazebo_ros2_control.so">
+            <parameters>$(find dr_description)/config/my_controllers.yaml</parameters>
+            <parameters>$(find dr_description)/config/gaz_ros2_ctl_use_sim.yaml</parameters>
         </plugin>
     </gazebo>
-    </xacro:macro>
 </robot>

Commit message: test per avere il namespace sul robot

File: dr_description/description/camera.xacro (robot description, xacro)
@@ -46,5 +46,8 @@
             </camera>
             <plugin name="camera_controller" filename="libgazebo_ros_camera.so">
-                <frame_name>camera_link_optical</frame_name>
+                <ros>
+                    <namespace>$(arg robot_namespace)</namespace>
+                </ros>
+                <frame_name>$(arg robot_namespace)/camera_link_optical</frame_name>
             </plugin>
         </sensor>

File: dr_description/description/depth_camera.xacro (robot description, xacro)
@@ -39,5 +39,8 @@
             </camera>
             <plugin name="camera_controller" filename="libgazebo_ros_camera.so">
-                <frame_name>camera_link_optical</frame_name>
+                <ros>
+                    <namespace>$(arg robot_namespace)</namespace>
+                </ros>
+                <frame_name>$(arg robot_namespace)/camera_link_optical</frame_name>
                 <min_depth>0.1</min_depth>
                 <max_depth>100.0</max_depth>

File: dr_description/description/depth_camera2.xacro (robot description, xacro)
@@ -39,5 +39,8 @@
             </camera>
             <plugin name="scanner_controller" filename="libgazebo_ros_camera.so">
-                <frame_name>scanner_link_optical</frame_name>
+                <ros>
+                    <namespace>$(arg robot_namespace)</namespace>
+                </ros>
+                <frame_name>$(arg robot_namespace)/scanner_link_optical</frame_name>
                 <min_depth>0.1</min_depth>
                 <max_depth>100.0</max_depth>

File: dr_description/description/face.xacro (robot description, xacro)
@@ -2,9 +2,9 @@
 <robot xmlns:xacro="http://www.ros.org/wiki/xacro" >
     <joint name="face_joint" type="fixed">
-        <parent link="chassis"/>
-        <child link="face_link"/>
+        <parent link="$(arg robot_namespace)/chassis"/>
+        <child link="$(arg robot_namespace)/face_link"/>
         <origin xyz="${chassis_length} 0 ${chassis_height/2}" rpy="0 0 0"/>
     </joint>
-    <link name="face_link">
+    <link name="$(arg robot_namespace)/face_link">
         <visual>
             <origin xyz="0 0.05 0.01" rpy="0 ${pi/2} 0"/>
@@ -29,5 +29,5 @@
         </visual>
     </link>
-    <gazebo reference="face_link">
+    <gazebo reference="$(arg robot_namespace)/face_link">
         <material>Gazebo/Black</material>
     </gazebo>

File: dr_description/description/gazebo_control.xacro (robot description, xacro)
@@ -3,7 +3,10 @@
     <gazebo>
         <plugin name="diff_drive" filename="libgazebo_ros_diff_drive.so">
+            <ros>
+                <namespace>$(arg robot_namespace)</namespace>
+            </ros>
             <!-- Wheel Information -->
             <left_joint>left_wheel_joint</left_joint>
-            <right_joint>right_wheel_joint</right_joint>
+            <right_joint>right_wheel_joint</right_wheel_joint>
             <wheel_separation>0.297</wheel_separation>
             <wheel_diameter>0.066</wheel_diameter>
@@ -12,6 +15,6 @@
             <max_wheel_acceleration>10.0</max_wheel_acceleration>
             <!-- Output -->
-            <odometry_frame>odom</odometry_frame>
-            <robot_base_frame>base_link</robot_base_frame>
+            <odometry_frame>$(arg robot_namespace)/odom</odometry_frame>
+            <robot_base_frame>$(arg robot_namespace)/base_link</robot_base_frame>
             <publish_odom>true</publish_odom>
             <publish_odom_tf>true</publish_odom_tf>

File: dr_description/description/lidar.xacro (robot description, xacro)
@@ -43,8 +43,9 @@
             <plugin name="laser_controller" filename="libgazebo_ros_ray_sensor.so">
                 <ros>
+                    <namespace>$(arg robot_namespace)</namespace>
                     <argument>~/out:=scan</argument>
                 </ros>
                 <output_type>sensor_msgs/LaserScan</output_type>
-                <frame_name>laser_frame</frame_name>
+                <frame_name>$(arg robot_namespace)/laser_frame</frame_name>
             </plugin>
         </sensor>

File: dr_description/description/robot.urdf.xacro (robot description, xacro)
@@ -1,7 +1,11 @@
 <?xml version="1.0"?>
-<robot xmlns:xacro="http://www.ros.org/wiki/xacro"  name="robot">
+<robot xmlns:xacro="http://www.ros.org/wiki/xacro" name="$(arg robot_namespace)">
+    <xacro:arg name="robot_namespace" default="minion"/>
     <xacro:arg name="use_ros2_control" default="true"/>
     <xacro:arg name="sim_mode" default="false"/>
     <xacro:include filename="robot_core.xacro" />
+    <xacro:include filename="lidar.xacro" />
+    <xacro:include filename="depth_camera.xacro" />
+    <xacro:include filename="depth_camera2.xacro" />
     <xacro:if value="$(arg use_ros2_control)">
         <xacro:include filename="ros2_control.xacro" />
@@ -10,8 +14,4 @@
         <xacro:include filename="gazebo_control.xacro" />
     </xacro:unless>
-    <xacro:include filename="lidar.xacro" />
-    <!-- <xacro:include filename="camera.xacro" /> -->
-    <xacro:include filename="depth_camera.xacro" />
-    <xacro:include filename="depth_camera2.xacro" />
     <!-- <xacro:include filename="face.xacro" /> -->
 </robot>

File: dr_description/description/ros2_control.xacro (robot description, xacro)
@@ -2,5 +2,5 @@
 <robot xmlns:xacro="http://www.ros.org/wiki/xacro">
     <xacro:unless value="$(arg sim_mode)">
-        <ros2_control name="RealRobot" type="system">
+        <ros2_control name="$(arg robot_namespace)_RealRobot" type="system">
             <hardware>
                 <plugin>diffdrive_arduino/DiffDriveArduinoHardware</plugin>
@@ -32,5 +32,5 @@
     </xacro:unless>
     <xacro:if value="$(arg sim_mode)">
-        <ros2_control name="GazeboSystem" type="system">
+        <ros2_control name="$(arg robot_namespace)_GazeboSystem" type="system">
             <hardware>
                 <plugin>gazebo_ros2_control/GazeboSystem</plugin>
@@ -56,6 +56,11 @@
     <gazebo>
         <plugin name="gazebo_ros2_control" filename="libgazebo_ros2_control.so">
+            <robot_param>robot_description</robot_param>
+            <robot_param_node>$(arg robot_namespace)</robot_param_node>
             <parameters>$(find dr_description)/config/my_controllers.yaml</parameters>
             <parameters>$(find dr_description)/config/gaz_ros2_ctl_use_sim.yaml</parameters>
+            <ros>
+                <namespace>$(arg robot_namespace)</namespace>
+            </ros>
         </plugin>
     </gazebo>
